Commit message: removed mock hardware

File: description/diffbot_ros2_control.xacro (robot description, xacro)
@@ -2,34 +2,26 @@
 <!-- included by, and macro expanded in, diffbot_urdf.xacro -->
 <robot xmlns:xacro="http://www.ros.org/wiki/xacro">
-  <xacro:macro name="diffbot_ros2_control" params="name prefix use_mock_hardware">
+  <xacro:macro name="diffbot_ros2_control" params="name prefix">
     <ros2_control name="${name}" type="system">
-      <xacro:unless value="${use_mock_hardware}">
-        <hardware>
-          <plugin>diffbot/DiffbotSystem</plugin>
-          <!-- used by both wheels -->
-          <param name="gpio_dev_name">/dev/gpiochip0</param>
-          <param name="pwm_chip_name">pwmchip0</param>
-          <!-- left wheel -->
-          <param name="left/dir_pin">17</param>
-          <param name="left/pwm_num">1</param>
-          <param name="left/pwm_rev">true</param>
-          <param name="left/enc_a_pin">3</param>
-          <param name="left/enc_b_pin">4</param>
-          <param name="left/enc_cpr">585</param>
-          <!-- right wheel -->
-          <param name="right/dir_pin">22</param>
-          <param name="right/pwm_num">0</param>
-          <param name="right/pwm_rev">false</param>
-          <param name="right/enc_a_pin">11</param>
-          <param name="right/enc_b_pin">9</param>
-          <param name="right/enc_cpr">585</param>
-        </hardware>
-      </xacro:unless>
-      <xacro:if value="${use_mock_hardware}">
-        <hardware>
-          <plugin>mock_components/GenericSystem</plugin>
-          <param name="calculate_dynamics">true</param>
-        </hardware>
-      </xacro:if>
+      <hardware>
+        <plugin>diffbot/DiffbotSystem</plugin>
+        <!-- used by both wheels -->
+        <param name="gpio_dev_name">/dev/gpiochip0</param>
+        <param name="pwm_chip_name">pwmchip0</param>
+        <!-- left wheel -->
+        <param name="left/dir_pin">17</param>
+        <param name="left/pwm_num">1</param>
+        <param name="left/pwm_rev">true</param>
+        <param name="left/enc_a_pin">3</param>
+        <param name="left/enc_b_pin">4</param>
+        <param name="left/enc_cpr">585</param>
+        <!-- right wheel -->
+        <param name="right/dir_pin">22</param>
+        <param name="right/pwm_num">0</param>
+        <param name="right/pwm_rev">false</param>
+        <param name="right/enc_a_pin">11</param>
+        <param name="right/enc_b_pin">9</param>
+        <param name="right/enc_cpr">585</param>
+      </hardware>
       <joint name="${prefix}left_wheel_joint">
         <command_interface name="velocity"/>

File: description/diffbot_urdf.xacro (robot description, xacro)
@@ -2,5 +2,4 @@
 <robot xmlns:xacro="http://www.ros.org/wiki/xacro" name="diffdrive_robot">
   <xacro:arg name="prefix" default=""/>
-  <xacro:arg name="use_mock_hardware" default="false"/>
   <!-- defines diffbot(prefix) -->
   <!-- uses the <material> definitions -->
@@ -8,7 +7,7 @@
   <!-- defines several <material> names -->
   <xacro:include filename="$(find diffbot)/description/material.xacro"/>
-  <!-- defines diffbot_ros2_control(name, prefix, use_mock_hardware) -->
+  <!-- defines diffbot_ros2_control(name, prefix) -->
   <xacro:include filename="$(find diffbot)/description/diffbot_ros2_control.xacro"/>
   <xacro:diffbot prefix="$(arg prefix)"/>
-  <xacro:diffbot_ros2_control name="Diffbot" prefix="$(arg prefix)" use_mock_hardware="$(arg use_mock_hardware)"/>
+  <xacro:diffbot_ros2_control name="Diffbot" prefix="$(arg prefix)"/>
 </robot>
