Commit message: removed material definitions

File: description/diffbot_description_urdf.xacro (robot description, xacro)
@@ -23,11 +23,4 @@
       </geometry>
     </collision>
-    <visual>
-      <origin xyz="0 0 ${base_height/2}" rpy="0 0 0"/>
-      <geometry>
-        <box size="${base_width} ${base_length} ${base_height}"/>
-      </geometry>
-      <material name="orange"/>
-    </visual>
     <inertial>
       <origin xyz="0 0 0" rpy="0 0 0"/>
@@ -55,11 +48,4 @@
         </geometry>
       </collision>
-      <visual>
-        <origin xyz="0 0 0" rpy="${PI/2} 0 0"/>
-        <geometry>
-          <cylinder length="${wheel_len}" radius="${wheel_radius}"/>
-        </geometry>
-        <material name="black"/>
-      </visual>
       <inertial>
         <origin xyz="0 0 0" rpy="${PI/2} 0 0"/>
@@ -87,11 +73,4 @@
         </geometry>
       </collision>
-      <visual>
-        <origin xyz="0 0 0" rpy="${PI/2} 0 0"/>
-        <geometry>
-          <cylinder length="${wheel_len}" radius="${wheel_radius}"/>
-        </geometry>
-        <material name="black"/>
-      </visual>
       <inertial>
         <origin xyz="0 0 0" rpy="${PI/2} 0 0"/>
@@ -116,11 +95,4 @@
         </geometry>
       </collision>
-      <visual>
-        <origin xyz="0 0 0" rpy="0 0 0"/>
-        <geometry>
-          <sphere radius="${caster_wheel_radius}"/>
-        </geometry>
-        <material name="white"/>
-      </visual>
       <inertial>
         <origin xyz="0 0 0" rpy="0 0 0"/>
@@ -145,11 +117,4 @@
         </geometry>
       </collision>
-      <visual>
-        <origin xyz="0 0 0" rpy="0 0 0"/>
-        <geometry>
-          <sphere radius="${caster_wheel_radius}"/>
-        </geometry>
-        <material name="white"/>
-      </visual>
       <inertial>
         <origin xyz="0 0 0" rpy="0 0 0"/>

File: description/diffbot_urdf.xacro (robot description, xacro)
@@ -3,8 +3,5 @@
   <xacro:arg name="prefix" default=""/>
   <!-- defines diffbot(prefix) -->
-  <!-- uses the <material> definitions -->
   <xacro:include filename="$(find diffbot)/description/diffbot_description_urdf.xacro"/>
-  <!-- defines several <material> names -->
-  <xacro:include filename="$(find diffbot)/description/material.xacro"/>
   <!-- defines diffbot_ros2_control(name, prefix) -->
   <xacro:include filename="$(find diffbot)/description/diffbot_ros2_control.xacro"/>

Commit message: removed caster wheels

File: description/diffbot_description_urdf.xacro (robot description, xacro)
@@ -12,6 +12,4 @@
   <xacro:property name="wheel_len" value="0.020" />
   <xacro:property name="wheel_radius" value="0.015" />
-  <xacro:property name="caster_wheel_mass" value="0.1" /> <!-- arbitrary value for caster wheel mass -->
-  <xacro:property name="caster_wheel_radius" value="0.015" />
   <xacro:property name="z_offset" value="-${base_height/2}" /> <!-- Space btw top of beam and the each joint -->
   <!-- Base Link -->
@@ -82,48 +80,4 @@
         </inertial>
       </link>
-    <joint name="${prefix}caster_frontal_wheel_joint" type="fixed">
-      <parent link="${prefix}base_link"/>
-      <child link="${prefix}caster_frontal_wheel"/>
-      <origin xyz="${base_width/2 - caster_wheel_radius} 0 ${z_offset}" rpy="0 0 0"/>
-    </joint>
-    <!-- caster frontal wheel Link -->
-    <link name="${prefix}caster_frontal_wheel">
-      <collision>
-        <origin xyz="0 0 0" rpy="0 0 0"/>
-        <geometry>
-          <sphere radius="${caster_wheel_radius}"/>
-        </geometry>
-      </collision>
-      <inertial>
-        <origin xyz="0 0 0" rpy="0 0 0"/>
-        <mass value="${caster_wheel_mass}"/>
-        <inertia
-          ixx="${caster_wheel_mass * 0.4 * (caster_wheel_radius * caster_wheel_radius)}" ixy="0.0" ixz="0.0"
-          iyy="${caster_wheel_mass * 0.4 * (caster_wheel_radius * caster_wheel_radius)}" iyz="0.0"
-          izz="${caster_wheel_mass * 0.4 * (caster_wheel_radius * caster_wheel_radius)}"/>
-        </inertial>
-      </link>
-    <joint name="${prefix}caster_rear_wheel_joint" type="fixed">
-      <parent link="${prefix}base_link"/>
-      <child link="${prefix}caster_rear_wheel"/>
-      <origin xyz="${-base_width/2 + caster_wheel_radius} 0 ${z_offset}" rpy="0 0 0"/>
-    </joint>
-    <!-- caster rear wheel Link -->
-    <link name="${prefix}caster_rear_wheel">
-      <collision>
-        <origin xyz="0 0 0" rpy="0 0 0"/>
-        <geometry>
-          <sphere radius="${caster_wheel_radius}"/>
-        </geometry>
-      </collision>
-      <inertial>
-        <origin xyz="0 0 0" rpy="0 0 0"/>
-        <mass value="${caster_wheel_mass}"/>
-        <inertia
-          ixx="${caster_wheel_mass * 0.4 * (caster_wheel_radius * caster_wheel_radius)}" ixy="0.0" ixz="0.0"
-          iyy="${caster_wheel_mass * 0.4 * (caster_wheel_radius * caster_wheel_radius)}" iyz="0.0"
-          izz="${caster_wheel_mass * 0.4 * (caster_wheel_radius * caster_wheel_radius)}"/>
-        </inertial>
-      </link>
   </xacro:macro>
 </robot>

Commit message: removed <inertial> tags

File: description/diffbot_description_urdf.xacro (robot description, xacro)
@@ -3,15 +3,11 @@
 <robot xmlns:xacro="http://www.ros.org/wiki/xacro">
   <xacro:macro name="diffbot" params="prefix">
-  <!-- Constants for robot dimensions -->
   <xacro:property name="PI" value="3.1415926535897931"/>
-  <xacro:property name="base_mass" value="0.3" /> <!-- arbitrary value for base mass -->
   <xacro:property name="base_width" value="0.1" />
   <xacro:property name="base_length" value="0.1" />
   <xacro:property name="base_height" value="0.05" />
-  <xacro:property name="wheel_mass" value="0.3" /> <!-- arbitrary value for wheel mass -->
   <xacro:property name="wheel_len" value="0.020" />
   <xacro:property name="wheel_radius" value="0.015" />
-  <xacro:property name="z_offset" value="-${base_height/2}" /> <!-- Space btw top of beam and the each joint -->
-  <!-- Base Link -->
+  <xacro:property name="z_offset" value="-${base_height/2}" />
   <link name="${prefix}base_link">
     <collision>
@@ -21,12 +17,4 @@
       </geometry>
     </collision>
-    <inertial>
-      <origin xyz="0 0 0" rpy="0 0 0"/>
-      <mass value="${base_mass}"/>
-      <inertia
-        ixx="${base_mass / 12.0 * (base_length*base_length + base_height*base_height)}" ixy="0.0" ixz="0.0"
-        iyy="${base_mass / 12.0 * (base_height*base_height + base_width*base_width)}" iyz="0.0"
-        izz="${base_mass / 12.0 * (base_width*base_width + base_length*base_length)}"/>
-      </inertial>
     </link>
     <joint name="${prefix}left_wheel_joint" type="continuous">
@@ -38,5 +26,4 @@
       <limit effort="100" velocity="1.0"/>
     </joint>
-    <!-- left wheel Link -->
     <link name="${prefix}left_wheel">
       <collision>
@@ -46,12 +33,4 @@
         </geometry>
       </collision>
-      <inertial>
-        <origin xyz="0 0 0" rpy="${PI/2} 0 0"/>
-        <mass value="${wheel_mass}"/>
-        <inertia
-          ixx="${wheel_mass / 12.0 * (3*wheel_radius*wheel_radius + wheel_len*wheel_len)}" ixy="0.0" ixz="0.0"
-          iyy="${wheel_mass / 12.0 * (3*wheel_radius*wheel_radius + wheel_len*wheel_len)}" iyz="0.0"
-          izz="${wheel_mass / 2.0 * wheel_radius*wheel_radius}"/>
-        </inertial>
       </link>
     <joint name="${prefix}right_wheel_joint" type="continuous">
@@ -63,5 +42,4 @@
       <limit effort="100" velocity="1.0"/>
     </joint>
-    <!-- right wheel Link -->
     <link name="${prefix}right_wheel">
       <collision>
@@ -71,12 +49,4 @@
         </geometry>
       </collision>
-      <inertial>
-        <origin xyz="0 0 0" rpy="${PI/2} 0 0"/>
-        <mass value="${wheel_mass}"/>
-        <inertia
-          ixx="${wheel_mass / 12.0 * (3*wheel_radius*wheel_radius + wheel_len*wheel_len)}" ixy="0.0" ixz="0.0"
-          iyy="${wheel_mass / 12.0 * (3*wheel_radius*wheel_radius + wheel_len*wheel_len)}" iyz="0.0"
-          izz="${wheel_mass / 2.0 * wheel_radius*wheel_radius}"/>
-        </inertial>
       </link>
   </xacro:macro>

Commit message: removed <collision> elements

File: description/diffbot_description_urdf.xacro (robot description, xacro)
@@ -3,19 +3,8 @@
 <robot xmlns:xacro="http://www.ros.org/wiki/xacro">
   <xacro:macro name="diffbot" params="prefix">
-  <xacro:property name="PI" value="3.1415926535897931"/>
-  <xacro:property name="base_width" value="0.1" />
-  <xacro:property name="base_length" value="0.1" />
-  <xacro:property name="base_height" value="0.05" />
-  <xacro:property name="wheel_len" value="0.020" />
-  <xacro:property name="wheel_radius" value="0.015" />
-  <xacro:property name="z_offset" value="-${base_height/2}" />
-  <link name="${prefix}base_link">
-    <collision>
-      <origin xyz="0 0 0" rpy="0 0 0"/>
-      <geometry>
-        <box size="${base_width} ${base_length} ${base_height}"/>
-      </geometry>
-    </collision>
-    </link>
+    <xacro:property name="base_width" value="0.1"/>
+    <xacro:property name="base_height" value="0.05"/>
+    <xacro:property name="z_offset" value="-${base_height/2}"/>
+    <link name="${prefix}base_link"/>
     <joint name="${prefix}left_wheel_joint" type="continuous">
       <parent link="${prefix}base_link"/>
@@ -26,12 +15,5 @@
       <limit effort="100" velocity="1.0"/>
     </joint>
-    <link name="${prefix}left_wheel">
-      <collision>
-        <origin xyz="0 0 0" rpy="${PI/2} 0 0"/>
-        <geometry>
-          <cylinder length="${wheel_len}" radius="${wheel_radius}"/>
-        </geometry>
-      </collision>
-      </link>
+    <link name="${prefix}left_wheel"/>
     <joint name="${prefix}right_wheel_joint" type="continuous">
       <parent link="${prefix}base_link"/>
@@ -42,12 +24,5 @@
       <limit effort="100" velocity="1.0"/>
     </joint>
-    <link name="${prefix}right_wheel">
-      <collision>
-        <origin xyz="0 0 0" rpy="${PI/2} 0 0"/>
-        <geometry>
-          <cylinder length="${wheel_len}" radius="${wheel_radius}"/>
-        </geometry>
-      </collision>
-      </link>
+    <link name="${prefix}right_wheel"/>
   </xacro:macro>
 </robot>

Commit message: removed remaining simulator-required stuff from urdf

File: description/diffbot_description_urdf.xacro (robot description, xacro)
@@ -3,15 +3,8 @@
 <robot xmlns:xacro="http://www.ros.org/wiki/xacro">
   <xacro:macro name="diffbot" params="prefix">
-    <xacro:property name="base_width" value="0.1"/>
-    <xacro:property name="base_height" value="0.05"/>
-    <xacro:property name="z_offset" value="-${base_height/2}"/>
     <link name="${prefix}base_link"/>
     <joint name="${prefix}left_wheel_joint" type="continuous">
       <parent link="${prefix}base_link"/>
       <child link="${prefix}left_wheel"/>
-      <origin xyz="0 -${base_width/2} ${z_offset}" rpy="0 0 0"/>
-      <axis xyz="0 1 0"/>
-      <dynamics damping="0.2"/>
-      <limit effort="100" velocity="1.0"/>
     </joint>
     <link name="${prefix}left_wheel"/>
@@ -19,8 +12,4 @@
       <parent link="${prefix}base_link"/>
       <child link="${prefix}right_wheel"/>
-      <origin xyz="0 ${base_width/2} ${z_offset}" rpy="0 0 0"/>
-      <axis xyz="0 1 0"/>
-      <dynamics damping="0.2"/>
-      <limit effort="100" velocity="1.0"/>
     </joint>
     <link name="${prefix}right_wheel"/>

Commit message: adjust wheel joints for rviz2
Move the wheel origins left and right so they are in the correct
positions and the wheels rotate in the correct directions.

File: description/diffbot_description_urdf.xacro (robot description, xacro)
@@ -3,8 +3,20 @@
 <robot xmlns:xacro="http://www.ros.org/wiki/xacro">
   <xacro:macro name="diffbot" params="prefix">
+    /!-- matches wheel_separation in diffbot_controllers.yaml -->
+    <xacro:property name="track" value="0.154" />
     <link name="${prefix}base_link"/>
     <joint name="${prefix}left_wheel_joint" type="continuous">
       <parent link="${prefix}base_link"/>
       <child link="${prefix}left_wheel"/>
+      <!-- These are only used when viewing the /tf topic using rviz2; they
+      make it so the wheel rotation looks correct. Driving the robot works
+      fine without them. +X is forward, +Y is left, and +Z is up. The origin
+      xyz is how to get from the parent to child origin, so positive Y means
+      to the left. Origin rpy is zero, so +X is still forward and +Y is still
+      left. Not sure how to interpret the axis vector but this makes it look
+      correct in rviz2.
+      -->
+      <origin xyz="0 +${track/2} 0" rpy="0 0 0"/>
+      <axis xyz="0 1 0"/>
     </joint>
     <link name="${prefix}left_wheel"/>
@@ -12,4 +24,6 @@
       <parent link="${prefix}base_link"/>
       <child link="${prefix}right_wheel"/>
+      <origin xyz="0 -${track/2} 0" rpy="0 0 0"/>
+      <axis xyz="0 1 0"/>
     </joint>
     <link name="${prefix}right_wheel"/>

File: description/diffbot_urdf.xacro (robot description, xacro)
@@ -2,7 +2,13 @@
 <robot xmlns:xacro="http://www.ros.org/wiki/xacro" name="diffdrive_robot">
   <xacro:arg name="prefix" default=""/>
-  <!-- defines diffbot(prefix) -->
+  <!--
+    defines diffbot(prefix)
+    links and joints
+  -->
   <xacro:include filename="$(find diffbot)/description/diffbot_description_urdf.xacro"/>
-  <!-- defines diffbot_ros2_control(name, prefix) -->
+  <!--
+    defines diffbot_ros2_control(name, prefix)
+    things required for ros2_control
+  -->
   <xacro:include filename="$(find diffbot)/description/diffbot_ros2_control.xacro"/>
   <xacro:diffbot prefix="$(arg prefix)"/>

Commit message: added base_footprint and laser links
Also turned the wheel origins so they rotate around Z.
Removed "prefix" from all the xacros.
Less logging from diffbot_system as it runs.

File: description/diffbot_description_urdf.xacro (robot description, xacro)
@@ -2,30 +2,47 @@
 <!-- included by, and macro expanded in, diffbot_urdf.xacro -->
 <robot xmlns:xacro="http://www.ros.org/wiki/xacro">
-  <xacro:macro name="diffbot" params="prefix">
-    /!-- matches wheel_separation in diffbot_controllers.yaml -->
+  <xacro:macro name="diffbot">
+    <!-- matches wheel_separation in diffbot_controllers.yaml -->
     <xacro:property name="track" value="0.154" />
-    <link name="${prefix}base_link"/>
-    <joint name="${prefix}left_wheel_joint" type="continuous">
-      <parent link="${prefix}base_link"/>
-      <child link="${prefix}left_wheel"/>
+    <link name="base_link"/>
+    <!-- slam_toolbox seems to want "base_footprint"; make it the same as
+    base_link. It could probably be done with a slam_toolbox parameter, but
+    there should really be a base_footprint anyway. -->
+    <joint name="base_footprint_joint" type="fixed">
+      <parent link="base_link"/>
+      <child link="base_footprint"/>
+      <origin xyz="0 0 0" rpy="0 0 0"/>
+    </joint>
+    <link name="base_footprint"/>
+    <!-- RPLidar might want "laser" link; make it the same as "base_link" but
+    rotated so they have the same forward direction. It should be raised up
+    a bit, but that doesn't really matter yet. -->
+    <joint name="laser_joint" type="fixed">
+      <parent link="base_link"/>
+      <child link="laser"/>
+      <origin xyz="0 0 0" rpy="0 0 ${pi}"/>
+    </joint>
+    <link name="laser"/>
+    <joint name="left_wheel_joint" type="continuous">
+      <parent link="base_link"/>
+      <child link="left_wheel"/>
       <!-- These are only used when viewing the /tf topic using rviz2; they
       make it so the wheel rotation looks correct. Driving the robot works
-      fine without them. +X is forward, +Y is left, and +Z is up. The origin
-      xyz is how to get from the parent to child origin, so positive Y means
-      to the left. Origin rpy is zero, so +X is still forward and +Y is still
-      left. Not sure how to interpret the axis vector but this makes it look
-      correct in rviz2.
-      -->
-      <origin xyz="0 +${track/2} 0" rpy="0 0 0"/>
-      <axis xyz="0 1 0"/>
+      fine without them. See http://wiki.ros.org/urdf/XML/joint.
+      +X is forward, +Y is left, and +Z is up. The origin xyz is how to get
+      from the parent to child origin, so positive Y means to the left. To
+      make the wheel rotate around Z, "roll" the origin counterclockwise
+      (negative) 180 degrees. -->
+      <origin xyz="0 +${track/2} 0" rpy="-${pi/2} 0 0"/>
+      <axis xyz="0 0 +1"/>
     </joint>
-    <link name="${prefix}left_wheel"/>
-    <joint name="${prefix}right_wheel_joint" type="continuous">
-      <parent link="${prefix}base_link"/>
-      <child link="${prefix}right_wheel"/>
-      <origin xyz="0 -${track/2} 0" rpy="0 0 0"/>
-      <axis xyz="0 1 0"/>
+    <link name="left_wheel"/>
+    <joint name="right_wheel_joint" type="continuous">
+      <parent link="base_link"/>
+      <child link="right_wheel"/>
+      <origin xyz="0 -${track/2} 0" rpy="+${pi/2} 0 0"/>
+      <axis xyz="0 0 -1"/>
     </joint>
-    <link name="${prefix}right_wheel"/>
+    <link name="right_wheel"/>
   </xacro:macro>
 </robot>

File: description/diffbot_ros2_control.xacro (robot description, xacro)
@@ -2,5 +2,5 @@
 <!-- included by, and macro expanded in, diffbot_urdf.xacro -->
 <robot xmlns:xacro="http://www.ros.org/wiki/xacro">
-  <xacro:macro name="diffbot_ros2_control" params="name prefix">
+  <xacro:macro name="diffbot_ros2_control" params="name">
     <ros2_control name="${name}" type="system">
       <hardware>
@@ -24,10 +24,10 @@
         <param name="right/enc_cpr">585</param>
       </hardware>
-      <joint name="${prefix}left_wheel_joint">
+      <joint name="left_wheel_joint">
         <command_interface name="velocity"/>
         <state_interface name="position"/>
         <state_interface name="velocity"/>
       </joint>
-      <joint name="${prefix}right_wheel_joint">
+      <joint name="right_wheel_joint">
         <command_interface name="velocity"/>
         <state_interface name="position"/>

File: description/diffbot_urdf.xacro (robot description, xacro)
@@ -1,16 +1,15 @@
 <?xml version="1.0"?>
 <robot xmlns:xacro="http://www.ros.org/wiki/xacro" name="diffdrive_robot">
-  <xacro:arg name="prefix" default=""/>
   <!--
-    defines diffbot(prefix)
+    defines diffbot()
     links and joints
   -->
   <xacro:include filename="$(find diffbot)/description/diffbot_description_urdf.xacro"/>
   <!--
-    defines diffbot_ros2_control(name, prefix)
+    defines diffbot_ros2_control(name)
     things required for ros2_control
   -->
   <xacro:include filename="$(find diffbot)/description/diffbot_ros2_control.xacro"/>
-  <xacro:diffbot prefix="$(arg prefix)"/>
-  <xacro:diffbot_ros2_control name="Diffbot" prefix="$(arg prefix)"/>
+  <xacro:diffbot/>
+  <xacro:diffbot_ros2_control name="Diffbot"/>
 </robot>
