Commit message: renaming from diffbot to rosbot in progress

File: description/rosbot_description_urdf.xacro (robot description, xacro)
@@ -1,7 +1,7 @@
 <?xml version="1.0"?>
-<!-- included by, and macro expanded in, diffbot_urdf.xacro -->
+<!-- included by, and macro expanded in, rosbot_urdf.xacro -->
 <robot xmlns:xacro="http://www.ros.org/wiki/xacro">
-  <xacro:macro name="diffbot">
-    <!-- matches wheel_separation in diffbot_controllers.yaml -->
+  <xacro:macro name="rosbot">
+    <!-- matches wheel_separation in rosbot_controllers.yaml -->
     <xacro:property name="track" value="0.154" />
     <link name="base_link"/>

File: description/rosbot_ros2_control.xacro (robot description, xacro)
@@ -1,9 +1,9 @@
 <?xml version="1.0"?>
-<!-- included by, and macro expanded in, diffbot_urdf.xacro -->
+<!-- included by, and macro expanded in, rosbot_urdf.xacro -->
 <robot xmlns:xacro="http://www.ros.org/wiki/xacro">
-  <xacro:macro name="diffbot_ros2_control" params="name">
+  <xacro:macro name="rosbot_ros2_control" params="name">
     <ros2_control name="${name}" type="system">
       <hardware>
-        <plugin>diffbot/DiffbotSystem</plugin>
+        <plugin>rosbot/RosBotSystem</plugin>
         <!-- used by both wheels -->
         <param name="ser_dev_name">/dev/ttyAMA0</param>
